Commit message: robot view

File: description/robot_core.xacro (robot description, xacro)
@@ -1,17 +1,111 @@
 <?xml version="1.0"?>
-<robot xmlns:xacro="http://www.ros.org/wiki/xacro" >
+<robot xmlns:xacro="http://www.ros.org/wiki/xacro">
+    <xacro:include filename="inertial_macros.xacro"/>
     <material name="white">
-    	<color rgba="1 1 1 1" />
+    	<color rgba="1 1 1 1"/>
     </material>
     <material name="orange">
-    	<color rgba="1 0.3 0.1 1" />
+    	<color rgba="1 0.3 0.1 1"/>
     </material>
     <material name="blue">
-    	<color rgba="0.2 0.2 1 1" />
+    	<color rgba="0.2 0.2 1 1"/>
     </material>
     <material name="black">
-    	<color rgba="0 0 0 1" />
+    	<color rgba="0 0 0 1"/>
     </material>
+    <!-- BASE_LINK -->
     <link name="base_link">
     </link>
+    <!-- CHASSIS -->
+    <link name="chassis">
+    	<visual>
+    	    <origin xyz="0.15 0 0.075"/>
+    	    <geometry>
+    	    	<box size="0.3 0.3 0.15"/>
+    	    </geometry>
+    	    <material name="orange"/>
+    	</visual>
+    	<collision>
+    	    <origin xyz="0.15 0 0.075"/>
+    	    <geometry>
+    	    	<box size="0.3 0.3 0.15"/>
+    	    </geometry>
+    	</collision>
+    	<xacro:inertial_box mass="0.5" x ="0.3" y="0.3" z="0.15">
+    	    <origin xyz="0.15 0 0" rpy="0 0 0"/>
+    	</xacro:inertial_box>
+    </link>
+    <joint name="chassis_joint" type="fixed">
+    	<parent link="base_link"/>
+    	<child link="chassis"/>
+    	<origin xyz="-0.1 0 0"/>
+    </joint>
+    <!-- LEFT_WHEEL -->
+    <link name="left_wheel">
+    	<visual>
+    	    <geometry>
+    	        <cylinder radius="0.05" length="0.04"/>
+    	    </geometry>
+    	    <material name="black"/>
+    	</visual>
+    	<collision>
+    	    <geometry>
+    	        <cylinder radius="0.05" length="0.04"/>
+    	    </geometry>
+    	</collision>
+    	<xacro:inertial_cylinder mass="0.1" length="0.04" radius="0.05">
+    	    <origin xyz="0 0 0" rpy="0 0 0"/>
+    	</xacro:inertial_cylinder>
+    </link>
+    <joint name="left_wheel_joint" type="continuous">
+    	<parent link="base_link"/>
+    	<child link="left_wheel"/>
+    	<origin xyz="0 0.175 0" rpy="-${pi/2} 0 0"/>
+    	<axis xyz="0 0 1"/>
+    </joint>
+    <!-- RIGHT_WHEEL -->
+    <link name="right_wheel">
+    	<visual>
+    	    <geometry>
+    	        <cylinder radius="0.05" length="0.04"/>
+    	    </geometry>
+    	    <material name="black"/>
+    	</visual>
+    	<collision>
+    	    <geometry>
+    	        <cylinder radius="0.05" length="0.04"/>
+    	    </geometry>
+    	</collision>
+    	<xacro:inertial_cylinder mass="0.1" length="0.04" radius="0.05">
+    	    <origin xyz="0 0 0" rpy="0 0 0"/>
+    	</xacro:inertial_cylinder>
+    </link>
+    <joint name="right_wheel_joint" type="continuous">
+    	<parent link="base_link"/>
+    	<child link="right_wheel"/>
+    	<origin xyz="0 -0.175 0" rpy="${pi/2} 0 0"/>
+    	<axis xyz="0 0 -1"/>
+    </joint>
+    <!-- CASTER WHEEL -->
+    <link name="caster_wheel">
+        <visual>
+            <geometry>
+    	        <sphere radius="0.05"/>
+    	    </geometry>
+    	    <material name="black"/>
+    	</visual>
+    	<collision>
+            <geometry>
+    	        <sphere radius="0.05"/>
+    	    </geometry>
+    	</collision>
+    	<xacro:inertial_sphere mass="0.1" radius="0.05">
+    	    <origin xyz="0 0 0" rpy="0 0 0"/>
+    	</xacro:inertial_sphere>
+    </link>
+    <joint name="caster_wheel_joint" type="fixed">
+        <parent link="chassis"/>
+        <child link="caster_wheel"/>
+        <origin xyz="0.24 0 0"/>
+    </joint>
 </robot>
