Commit message: gazebo world

File: description/robot.urdf.xacro (robot description, xacro)
@@ -1,4 +1,5 @@
 <?xml version="1.0"?>
 <robot xmlns:xacro="http://www.ros.org/wiki/xacro"  name="robot">
-    <xacro:include filename="robot_core.xacro" />
+    <xacro:include filename="robot_core.xacro"/>
+    <xacro:include filename="gazebo_control.xacro"/>
 </robot>

File: description/robot_core.xacro (robot description, xacro)
@@ -36,4 +36,7 @@
     	</xacro:inertial_box>
     </link>
+    <gazebo reference="chassis">
+        <material>Gazebo/Orange</material>
+    </gazebo>
     <joint name="chassis_joint" type="fixed">
     	<parent link="base_link"/>
@@ -58,4 +61,7 @@
     	</xacro:inertial_cylinder>
     </link>
+    <gazebo reference="left_wheel">
+        <material>Gazebo/Black</material>
+    </gazebo>
     <joint name="left_wheel_joint" type="continuous">
     	<parent link="base_link"/>
@@ -81,4 +87,7 @@
     	</xacro:inertial_cylinder>
     </link>
+    <gazebo reference="right_wheel">
+        <material>Gazebo/Black</material>
+    </gazebo>
     <joint name="right_wheel_joint" type="continuous">
     	<parent link="base_link"/>
@@ -104,4 +113,9 @@
     	</xacro:inertial_sphere>
     </link>
+    <gazebo reference="caster_wheel">
+        <material>Gazebo/Black</material>
+        <mu1 value="0.001"/>
+        <mu2 value="0.001"/>
+    </gazebo>
     <joint name="caster_wheel_joint" type="fixed">
         <parent link="chassis"/>

Commit message: lidar, camera, depth_camera

File: description/robot.urdf.xacro (robot description, xacro)
@@ -3,3 +3,6 @@
     <xacro:include filename="robot_core.xacro"/>
     <xacro:include filename="gazebo_control.xacro"/>
+    <!-- <xacro:include filename="lidar.xacro"/> -->
+    <!-- <xacro:include filename="camera.xacro"/> -->
+    <xacro:include filename="depth_camera.xacro"/>
 </robot>

File: description/robot_core.xacro (robot description, xacro)
@@ -4,4 +4,7 @@
     <material name="white">
     	<color rgba="1 1 1 1"/>
+    </material>
+    <material name="red">
+    	<color rgba="1 0 0 1"/>
     </material>
     <material name="orange">

Commit message: lidar, camera, slam, joystick

File: description/robot.urdf.xacro (robot description, xacro)
@@ -3,6 +3,7 @@
     <xacro:include filename="robot_core.xacro"/>
     <xacro:include filename="gazebo_control.xacro"/>
-    <!-- <xacro:include filename="lidar.xacro"/> -->
+    <!-- <xacro:include filename="ros2_control.xacro"/> -->
+    <xacro:include filename="lidar.xacro"/>
     <!-- <xacro:include filename="camera.xacro"/> -->
-    <xacro:include filename="depth_camera.xacro"/>
+    <!-- <xacro:include filename="depth_camera.xacro"/> -->
 </robot>

File: description/robot_core.xacro (robot description, xacro)
@@ -20,4 +20,11 @@
     <link name="base_link">
     </link>
+	<link name="base_footprint">
+	</link>
+	<joint name="base_footprint_joint" type="fixed">
+		<parent link="base_link"/>
+		<child link="base_footprint"/>
+		<origin xyz="0 0 0" rpy="0 0 0"/>
+	</joint>
     <!-- CHASSIS -->
     <link name="chassis">
