Commit message: squared robot -> tb2; add imu

File: description/depth_camera.xacro (robot description, xacro)
@@ -1,47 +1,47 @@
 <?xml version="1.0"?>
-<robot xmlns:xacro="http://www.ros.org/wiki/xacro" >
-    <joint name="camera_joint" type="fixed">
-        <parent link="camera_box"/>
-        <child link="camera_link"/>
-        <origin xyz="0.165 0 0" rpy="0 0 0"/>
-    </joint>
-    <link name="camera_link">
-        <visual>
-            <geometry>
-                <box size="0.01 0.04 0.04"/>
-            </geometry>
-            <material name="black"/>
-        </visual>
-    </link>
-    <joint name="camera_optical_joint" type="fixed">
-        <parent link="camera_link"/>
-        <child link="camera_link_optical"/>
-        <origin xyz="0 0 0" rpy="${-pi/2} 0 ${-pi/2}"/>
-    </joint>
-    <link name="camera_link_optical"></link>
-    <gazebo reference="camera_link">
-        <material>Gazebo/Black</material>
-        <sensor name="camera" type="depth">
-            <pose> 0 0 0 0 0 0 </pose>
-            <visualize>true</visualize>
-            <update_rate>20</update_rate>
-            <camera>
-                <horizontal_fov>1.089</horizontal_fov>
-                <image>
-                    <format>B8G8R8</format>
-                    <width>640</width>
-                    <height>480</height>
-                </image>
-                <clip>
-                    <near>0.05</near>
-                    <far>20</far>
-                </clip>
-            </camera>
-            <plugin name="camera_controller" filename="libgazebo_ros_camera.so">
-                <frame_name>camera_link_optical</frame_name>
-                <min_depth>0.1</min_depth>
-                <max_depth>20.0</max_depth>
-            </plugin>
-        </sensor>
-    </gazebo>
+<robot xmlns:xacro="http://www.ros.org/wiki/xacro">
+            <joint name="camera_joint" type="fixed">
+                <parent link="chassis" />
+                <child link="camera_link" />
+                <origin xyz="0.127 0 0" rpy="0 0 0" />
+            </joint>
+            <link name="camera_link">
+                <visual>
+                    <geometry>
+                        <box size="0.1 0.04 0.04" />
+                    </geometry>
+                    <material name="black" />
+                </visual>
+            </link>
+            <joint name="camera_optical_joint" type="fixed">
+                <parent link="camera_link" />
+                <child link="camera_link_optical" />
+                <origin xyz="0 0 0" rpy="${-pi/2} 0 ${-pi/2}" />
+            </joint>
+            <link name="camera_link_optical"></link>
+            <gazebo reference="camera_link">
+                <material>Gazebo/Black</material>
+                <sensor name="camera" type="depth">
+                    <pose> 0 0 0 0 0 0 </pose>
+                    <visualize>true</visualize>
+                    <update_rate>30</update_rate>
+                    <camera>
+                        <horizontal_fov>1.089</horizontal_fov>
+                        <image>
+                            <format>B8G8R8</format>
+                            <width>640</width>
+                            <height>480</height>
+                        </image>
+                        <clip>
+                            <near>0.05</near>
+                            <far>8.0</far>
+                        </clip>
+                    </camera>
+                    <plugin name="camera_controller" filename="libgazebo_ros_camera.so">
+                        <frame_name>camera_link_optical</frame_name>
+                        <min_depth>0.1</min_depth>
+                        <max_depth>100.0</max_depth>
+                    </plugin>
+                </sensor>
+            </gazebo>
 </robot>

File: description/gazebo_control.xacro (robot description, xacro)
@@ -3,22 +3,21 @@
     <gazebo>
         <plugin name="diff_drive" filename="libgazebo_ros_diff_drive.so">
-            <!-- <ros>
+            <ros>
                 <namespace>/robot</namespace>
-            </ros> -->
+            </ros>
             <!-- WHEEL INFORMATION -->
             <left_joint>left_wheel_joint</left_joint>
             <right_joint>right_wheel_joint</right_joint>
-            <wheel_separation>0.36</wheel_separation>
-            <wheel_diameter>0.1</wheel_diameter>
+            <wheel_separation>0.314</wheel_separation>
+            <wheel_diameter>0.08</wheel_diameter>
             <!-- LIMITS -->
             <max_wheel_torque>200</max_wheel_torque>
             <max_wheel_acceleration>10.0</max_wheel_acceleration>
             <!-- OUTPUT -->
+            <odometry_frame>odom</odometry_frame>
+            <robot_base_frame>base_footprint</robot_base_frame>
             <publish_odom>true</publish_odom>
             <publish_odom_tf>true</publish_odom_tf>
             <publish_wheel_tf>true</publish_wheel_tf>
-            <odometry_topic>odom</odometry_topic>
-            <odometry_frame>odom</odometry_frame>
-            <robot_base_frame>base_footprint</robot_base_frame>
         </plugin>
     </gazebo>

File: description/lidar.xacro (robot description, xacro)
@@ -46,7 +46,7 @@
     </gazebo>
     <joint name="laser_joint" type="fixed">
-        <parent link="base_link"/>
+        <parent link="chassis"/>
         <child link="laser_frame"/>
-        <origin xyz="0 0 0.1" rpy="0 0 0"/>
+        <origin xyz="0 0 0.230" rpy="0 0 0"/>
     </joint>
 </robot>

File: description/robot.urdf.xacro (robot description, xacro)
@@ -1,7 +1,8 @@
 <?xml version="1.0"?>
-<robot xmlns:xacro="http://www.ros.org/wiki/xacro"  name="dyn">
+<robot xmlns:xacro="http://www.ros.org/wiki/xacro"  name="robot">
     <xacro:include filename="robot_core.xacro"/>
     <xacro:include filename="gazebo_control.xacro"/>
     <xacro:include filename="lidar.xacro"/>
     <xacro:include filename="depth_camera.xacro"/>
+    <xacro:include filename="imu.xacro"/>
 </robot>

File: description/robot_core.xacro (robot description, xacro)
@@ -1,68 +1,56 @@
 <?xml version="1.0"?>
 <robot xmlns:xacro="http://www.ros.org/wiki/xacro">
-    <xacro:include filename="inertial_macros.xacro"/>
-	<!-- COLORS -->
+	<xacro:include filename="inertial_macros.xacro" />
+    <material name="white">
+		<color rgba="1 1 1 1" />
+    </material>
+    <material name="red">
+		<color rgba="1 0 0 1" />
+    </material>
     <material name="orange">
-    	<color rgba="1 0.3 0.1 0.5"/>
+		<color rgba="1 0.3 0.1 1" />
+    </material>
+    <material name="blue">
+		<color rgba="0.2 0.2 1 1" />
     </material>
     <material name="black">
-    	<color rgba="0 0 0 1"/>
+		<color rgba="0 0 0 1" />
     </material>
-    <!-- BASE_FOOTPRINT -->
+    <!-- BASE_LINK -->
+    <link name="base_link">
+    </link>
 	<link name="base_footprint">
 	</link>
-	<!-- BASE_LINK -->
-    <link name="base_link">
-		<visual>
-    	    <origin xyz="0 0 0"/>
+	<joint name="base_footprint_joint" type="fixed">
+		<parent link="base_footprint" />
+		<child  link="base_link" />
+		<origin xyz="0 0 0" rpy="0 0 0" />
+	</joint>
+    <!-- CHASSIS -->
+    <link name="chassis">
+    	<visual>
+			<origin xyz="0 0 0" />
     	    <geometry>
-    	    	<box size="0.32 0.32 0.16"/>
+				<cylinder radius="0.177" length="0.420" />
     	    </geometry>
-    	    <material name="orange"/>
+			<material name="orange" />
     	</visual>
     	<collision>
-    	    <origin xyz="0 0 0"/>
+			<origin xyz="0 0 0" />
     	    <geometry>
-    	    	<box size="0.32 0.32 0.16"/>
+				<cylinder radius="0.177" length="0.420" />
     	    </geometry>
     	</collision>
-    	<xacro:inertial_box mass="0.5" x="0.32" y="0.32" z="0.16">
-    	    <origin xyz="0 0 0" rpy="0 0 0"/>
-    	</xacro:inertial_box>
+    	<xacro:inertial_cylinder mass="0.5" length="0.420" radius="0.177">
+			<origin xyz="0 0 0" rpy="0 0 0" />
+    	</xacro:inertial_cylinder>
     </link>
-    <gazebo reference="base_link">
+    <gazebo reference="chassis">
         <material>Gazebo/Orange</material>
     </gazebo>
-    <joint name="base_link_joint" type="fixed">
-    	<parent link="base_footprint"/>
-    	<child link="base_link"/>
-    	<origin xyz="0 0 0.13"/>
-    </joint>
-	<!-- CAMERA_BOX -->
-	<link name="camera_box">
-		<visual>
-			<origin xyz="0 0 0"/>
-			<geometry>
-				<box size="0.32 0.32 0.32"/>
-			</geometry>
-			<material name="orange"/>
-		</visual>
-		<collision>
-			<origin xyz="0 0 0"/>
-			<geometry>
-				<box size="0.32 0.32 0.32"/>
-			</geometry>
-		</collision>
-		<!-- <xacro:inertial_box mass="0.5" x="0.32" y="0.32" z="0.32">
-    	    <origin xyz="0 0 0" rpy="0 0 0"/>
-    	</xacro:inertial_box> -->
-	</link>
-	<gazebo reference="camera_box">
-        <material>Gazebo/Orange</material>
-    </gazebo>
-    <joint name="camera_box_joint" type="fixed">
-    	<parent link="base_link"/>
-    	<child link="camera_box"/>
-    	<origin xyz="0 0 0.24"/>
+    <joint name="chassis_joint" type="fixed">
+		<parent link="base_link" />
+		<child link="chassis" />
+		<origin xyz="0 0 0" />
     </joint>
     <!-- LEFT_WHEEL -->
@@ -70,15 +58,15 @@
     	<visual>
     	    <geometry>
-    	        <cylinder radius="0.05" length="0.04"/>
+				<cylinder radius="0.04" length="0.04" />
     	    </geometry>
-    	    <material name="black"/>
+			<material name="black" />
     	</visual>
     	<collision>
     	    <geometry>
-    	        <cylinder radius="0.05" length="0.04"/>
+				<cylinder radius="0.04" length="0.04" />
     	    </geometry>
     	</collision>
-    	<xacro:inertial_cylinder mass="0.1" length="0.04" radius="0.05">
-    	    <origin xyz="0 0 0" rpy="0 0 0"/>
+    	<xacro:inertial_cylinder mass="0.1" length="0.04" radius="0.04">
+			<origin xyz="0 0 0" rpy="0 0 0" />
     	</xacro:inertial_cylinder>
     </link>
@@ -87,8 +75,8 @@
     </gazebo>
     <joint name="left_wheel_joint" type="continuous">
-    	<parent link="base_link"/>
-    	<child link="left_wheel"/>
-    	<origin xyz="-0.06 0.18 -0.08" rpy="-${pi/2} 0 0"/>
-    	<axis xyz="0 0 1"/>
+		<parent link="chassis" />
+		<child link="left_wheel" />
+		<origin xyz="0 0.157 -0.210" rpy="-${pi/2} 0 0" />
+		<axis xyz="0 0 1" />
     </joint>
     <!-- RIGHT_WHEEL -->
@@ -96,15 +84,15 @@
     	<visual>
     	    <geometry>
-    	        <cylinder radius="0.05" length="0.04"/>
+				<cylinder radius="0.04" length="0.04" />
     	    </geometry>
-    	    <material name="black"/>
+			<material name="black" />
     	</visual>
     	<collision>
     	    <geometry>
-    	        <cylinder radius="0.05" length="0.04"/>
+				<cylinder radius="0.04" length="0.04" />
     	    </geometry>
     	</collision>
-    	<xacro:inertial_cylinder mass="0.1" length="0.04" radius="0.05">
-    	    <origin xyz="0 0 0" rpy="0 0 0"/>
+    	<xacro:inertial_cylinder mass="0.1" length="0.04" radius="0.04">
+			<origin xyz="0 0 0" rpy="0 0 0" />
     	</xacro:inertial_cylinder>
     </link>
@@ -113,35 +101,61 @@
     </gazebo>
     <joint name="right_wheel_joint" type="continuous">
-    	<parent link="base_link"/>
-    	<child link="right_wheel"/>
-    	<origin xyz="-0.06 -0.18 -0.08" rpy="${pi/2} 0 0"/>
-    	<axis xyz="0 0 -1"/>
+		<parent link="chassis" />
+		<child link="right_wheel" />
+		<origin xyz="0 -0.157 -0.210" rpy="${pi/2} 0 0" />
+		<axis xyz="0 0 -1" />
     </joint>
     <!-- CASTER WHEEL -->
-    <link name="caster_wheel">
+    <link name="caster_wheel_forward">
         <visual>
             <geometry>
-    	        <sphere radius="0.05"/>
+				<sphere radius="0.04" />
     	    </geometry>
-    	    <material name="black"/>
+			<material name="black" />
     	</visual>
     	<collision>
             <geometry>
-    	        <sphere radius="0.05"/>
+				<sphere radius="0.04" />
     	    </geometry>
     	</collision>
-    	<xacro:inertial_sphere mass="0.1" radius="0.05">
-    	    <origin xyz="0 0 0" rpy="0 0 0"/>
+    	<xacro:inertial_sphere mass="0.1" radius="0.04">
+			<origin xyz="0 0 0" rpy="0 0 0" />
     	</xacro:inertial_sphere>
     </link>
-    <gazebo reference="caster_wheel">
+    <gazebo reference="caster_wheel_forward">
         <material>Gazebo/Black</material>
-        <mu1 value="0.001"/>
-        <mu2 value="0.001"/>
+		<mu1 value="0.001" />
+		<mu2 value="0.001" />
     </gazebo>
-    <joint name="caster_wheel_joint" type="fixed">
-        <parent link="base_link"/>
-        <child link="caster_wheel"/>
-        <origin xyz="0.1 0 -0.08"/>
+    <joint name="caster_wheel_forward_joint" type="fixed">
+		<parent link="chassis" />
+		<child link="caster_wheel_forward" />
+		<origin xyz="0.12 0 -0.210" />
     </joint>
+	<link name="caster_wheel_backward">
+		<visual>
+			<geometry>
+				<sphere radius="0.04" />
+			</geometry>
+			<material name="black" />
+		</visual>
+		<collision>
+			<geometry>
+				<sphere radius="0.04" />
+			</geometry>
+		</collision>
+		<xacro:inertial_sphere mass="0.1" radius="0.04">
+			<origin xyz="0 0 0" rpy="0 0 0" />
+		</xacro:inertial_sphere>
+	</link>
+	<gazebo reference="caster_wheel_backward">
+		<material>Gazebo/Black</material>
+		<mu1 value="0.001" />
+		<mu2 value="0.001" />
+	</gazebo>
+	<joint name="caster_wheel_backward_joint" type="fixed">
+		<parent link="chassis" />
+		<child link="caster_wheel_backward" />
+		<origin xyz="-0.12 0 -0.210" />
+	</joint>
 </robot>
